File: SolarTracker/kicad/solar-tracker.sch (KiCad schematic (older format))
At the start: 11 parts, among them J1 H-bridge1-connector, J2 H-bridge2-connector, U1 arduino_nano

Commit message: Devel
Parts:
- added J1: Power connector, symbol Conn_01x02
- added PWR1: +24V, symbol +24V
- added U2: DC-DC_Stepdown, symbol DC-DC_Stepdown
- J1: value H-bridge1-connector -> horiz actuator driver conn
- J2: value H-bridge2-connector -> vert actuator driver conn
Connections:
- net +12V: now also U2.2 (Vout)
- net GND: now also J1.1 (Pin_1), U2.1 (GND), U2.4 (GND)
- net verticalActuatorPwm: now reaches U1.D3 (#D3)
- net horizontalActuatorPwm: now reaches U1.D5 (#D5)
- new net +24V: J1.2 (Pin_2), PWR1.1 (+24V), U2.3 (VIN)
Changed lines of the file:
@@
 LIBS:valves
 LIBS:arduino
+LIBS:Zimprich
 LIBS:solar-tracker-cache
 EELAYER 25 0
@@
 P 6700 800
 F 0 "J1" H 6700 1100 50  0000 C CNN
-F 1 "H-bridge1-connector" V 6779 761 50  0000 C TNN
+F 1 "horiz actuator driver conn" V 6779 761 50  0000 C TNN
 F 2 "" H 6700 800 50  0001 C CNN
 F 3 "" H 6700 800 50  0001 C CNN
@@
 P 7900 800
 F 0 "J2" H 7900 1100 50  0000 C CNN
-F 1 "H-bridge2-connector" V 7979 761 50  0000 C TNN
+F 1 "vert actuator driver conn" V 7979 761 50  0000 C TNN
 F 2 "" H 7900 800 50  0001 C CNN
 F 3 "" H 7900 800 50  0001 C CNN
@@
 	0    -1   -1   0
 $EndComp
+$Comp
+L DC-DC_Stepdown U2
+U 1 1 5A6CE95B
+P 1350 1000
+F 0 "U2" H 1350 1200 60  0000 C BNN
+F 1 "DC-DC_Stepdown" H 1350 1000 16  0000 C CNN
+F 2 "" H 1350 1000 60  0000 C CNN
+F 3 "" H 1350 1000 60  0000 C CNN
+	1    1350 1000
+	1    0    0    -1
+$EndComp
+$Comp
+L GND #PWR?
+U 1 1 5A6CED94
+P 600 900
+F 0 "#PWR?" H 600 650 50  0001 C CNN
+F 1 "GND" H 600 750 50  0000 C CNN
+F 2 "" H 600 900 50  0001 C CNN
+F 3 "" H 600 900 50  0001 C CNN
+	1    600  900
+	1    0    0    -1
+$EndComp
+$Comp
+L GND #PWR?
+U 1 1 5A6CEDC3
+P 2000 900
+F 0 "#PWR?" H 2000 650 50  0001 C CNN
+F 1 "GND" H 2000 750 50  0000 C CNN
+F 2 "" H 2000 900 50  0001 C CNN
+F 3 "" H 2000 900 50  0001 C CNN
+	1    2000 900
+	1    0    0    -1
+$EndComp
+Wire Wire Line
+	2000 900  1700 900
+Wire Wire Line
+	600  900  1000 900
+$Comp
+L +12V #PWR?
+U 1 1 5A6CF160
+P 1800 1100
+F 0 "#PWR?" H 1800 950 50  0001 C CNN
+F 1 "+12V" H 1800 1240 50  0000 C CNN
+F 2 "" H 1800 1100 50  0001 C CNN
+F 3 "" H 1800 1100 50  0001 C CNN
+	1    1800 1100
+	-1   0    0    1
+$EndComp
+Wire Wire Line
+	1800 1100 1700 1100
+$Comp
+L +24V #PWR?
+U 1 1 5A6CF286
+P 850 1100
+F 0 "#PWR?" H 850 950 50  0001 C CNN
+F 1 "+24V" H 850 1240 50  0000 C CNN
+F 2 "" H 850 1100 50  0001 C CNN
+F 3 "" H 850 1100 50  0001 C CNN
+	1    850  1100
+	-1   0    0    1
+$EndComp
+Wire Wire Line
+	850  1100 1000 1100
+$Comp
+L Conn_01x02 J1
+U 1 1 5A6CFD2E
+P 2650 900
+F 0 "J1" H 2650 1000 50  0000 C CNN
+F 1 "Power connector" V 2750 800 50  0000 C CNN
+F 2 "" H 2650 900 50  0001 C CNN
+F 3 "" H 2650 900 50  0001 C CNN
+	1    2650 900
+	0    -1   -1   0
+$EndComp
+$Comp
+L +24V PWR1
+U 1 1 5A6D0C68
+P 2900 1200
+F 0 "PWR1" H 2900 1050 50  0001 C CNN
+F 1 "+24V" H 2900 1340 50  0000 C CNN
+F 2 "" H 2900 1200 50  0001 C CNN
+F 3 "" H 2900 1200 50  0001 C CNN
+	1    2900 1200
+	-1   0    0    1
+$EndComp
+$Comp
+L GND #PWR?
+U 1 1 5A6D0C9A
+P 2650 1200
+F 0 "#PWR?" H 2650 950 50  0001 C CNN
+F 1 "GND" H 2650 1050 50  0000 C CNN
+F 2 "" H 2650 1200 50  0001 C CNN
+F 3 "" H 2650 1200 50  0001 C CNN
+	1    2650 1200
+	1    0    0    -1
+$EndComp
+Wire Wire Line
+	2650 1100 2650 1200
+Wire Wire Line
+	2750 1100 2750 1200
+Wire Wire Line
+	2750 1200 2900 1200
+Text GLabel 5200 2100 2    60   Input ~ 0
+horizontalActuatorPwm
+Wire Wire Line
+	4850 2100 5200 2100
+Text GLabel 5200 2300 2    60   Input ~ 0
+verticalActuatorPwm
+Wire Wire Line
+	4850 2300 5200 2300
 $EndSCHEMATC

Commit message: kicad
Parts:
- removed PWR1: +24V, symbol +24V
- removed R1, R2, R3, R4: LDR07, Opto-Devices:Resistor_LDR_5.1x4.3_RM3.4, symbol LDR07
- removed R5, R6, R7, R8: R, symbol R
- added J1: To sensor, symbol Conn_01x06
- added U2: Wlan_ESP8266_mit_Pinnummern, MODULE, symbol Wlan_ESP8266_mit_Pinnummern
- U1: footprint DIL20 -> (none)
- renumbered J1 to J2, J2 to J3
Connections:
- net +5V: now also J2.1 (Pin_1), J2.4 (Pin_4), J3.1 (Pin_1), J3.4 (Pin_4), J1.1 (Pin_1)
- net GND: now also J2.6 (Pin_6), J3.6 (Pin_6), J1.2 (Pin_2)
- net horizontalActuatorPwm: now also J2.5 (Pin_5)
- net verticalActuatorPwm: now also J3.5 (Pin_5)
- net at U1.A0: now also J1.6 (Pin_6)
- net at U1.A1: now also J1.5 (Pin_5)
- net at U1.A2: now also J1.4 (Pin_4)
- net at U1.A3: now also J1.3 (Pin_3)
- net vertContractingDir: now reaches U1.D2
- net vertContractingDir: now also J3.2 (Pin_2)
- net vertExtendingDir: now reaches U1.D4
- net vertExtendingDir: now also J3.3 (Pin_3)
- net horizContractingDir: now reaches U1.D7
- net horizContractingDir: now also J2.2 (Pin_2)
- net horizExtendingDir: now reaches U1.D8
- net horizExtendingDir: now also J2.3 (Pin_3)
Other:
- moved on the sheet: J2, J3
